File: Schematics/_saved_Nigun.sch (KiCad schematic (older format))
At the start: 41 parts, among them J1 RF_INPUT, U1 ADRF6612, U2 SKY13373

Commit message: - Updated schematics - Added mini-circuits TC1-1-43A+ transformer to kicad library - Added AVX low-pass filter to lkicad ibrary
Parts:
- added C? (x2): 100pF, symbol C
- added T?: TC1-1-43A+, symbol TC1-1-43A+
Connections:
- net Earth: now also T?.6
- net at U1.4 (EXTVCOIN+): now also C?.1
- net at U1.5 (EXTVCOIN-): now also C?.1
- net at C?.1: now also T?.4
- new net: C?.2, T?.3
- new net: C?.2, T?.1
Other:
- note added: "02/10/2016"
- note added: "NIGUN - 1500-3000MHz RF downconverter for SDR"
Changed lines of the file:
@@
 	4600 2000 3750 2000
 Wire Wire Line
-	3750 1750 3750 2000
+	3750 2000 3750 1750
 Wire Wire Line
-	3000 1750 3750 1750
+	3750 1750 3000 1750
 Connection ~ 3100 1750
 Wire Wire Line
@@
 Connection ~ 2100 1750
 Wire Wire Line
-	3100 2350 3100 2050
-Wire Wire Line
-	1750 2350 4300 2350
+	3100 2350 1750 2350
 Wire Wire Line
 	2600 2050 2600 2350
@@
 	1750 2050 1750 2350
 Connection ~ 2100 2350
-Wire Wire Line
-	4600 2200 4300 2200
-Wire Wire Line
-	4300 2200 4300 2350
 Connection ~ 3100 2350
 Wire Wire Line
@@
 Wire Wire Line
 	3750 1450 3750 1300
-Wire Wire Line
-	4600 2400 3700 2400
 Connection ~ 6100 6200
 Connection ~ 6100 5900
@@
 Wire Wire Line
 	7300 6900 13850 6900
+$Comp
+L C C?
+U 1 1 57F058D1
+P 3200 2850
+F 0 "C?" H 3225 2950 50  0000 L CNN
+F 1 "100pF" H 3225 2750 50  0000 L CNN
+F 2 "" H 3238 2700 50  0000 C CNN
+F 3 "" H 3200 2850 50  0000 C CNN
+	1    3200 2850
+	0    1    1    0
+$EndComp
+$Comp
+L C C?
+U 1 1 57F058D7
+P 3200 2550
+F 0 "C?" H 3225 2650 50  0000 L CNN
+F 1 "100pF" H 3225 2450 50  0000 L CNN
+F 2 "" H 3238 2400 50  0000 C CNN
+F 3 "" H 3200 2550 50  0000 C CNN
+	1    3200 2550
+	0    1    1    0
+$EndComp
+$Comp
+L TC1-1-43A+ T?
+U 1 1 57F058DD
+P 2400 2500
+F 0 "T?" H 2400 2000 60  0000 C CNN
+F 1 "TC1-1-43A+" H 2400 2450 60  0000 C CNN
+F 2 "" H 2400 2500 60  0000 C CNN
+F 3 "" H 2400 2500 60  0000 C CNN
+	1    2400 2500
+	1    0    0    -1
+$EndComp
+$Comp
+L Earth #PWR?
+U 1 1 57F058E3
+P 2100 2850
+F 0 "#PWR?" H 2100 2600 50  0001 C CNN
+F 1 "Earth" H 2100 2700 50  0001 C CNN
+F 2 "" H 2100 2850 50  0000 C CNN
+F 3 "" H 2100 2850 50  0000 C CNN
+	1    2100 2850
+	1    0    0    -1
+$EndComp
+Wire Wire Line
+	3050 2850 2700 2850
+Wire Wire Line
+	3050 2550 2700 2550
+Wire Wire Line
+	2700 2550 2700 2700
+Wire Wire Line
+	4600 2600 3650 2600
+Wire Wire Line
+	3650 2600 3650 2850
+Wire Wire Line
+	3650 2850 3350 2850
+Wire Wire Line
+	4600 2400 3350 2400
+Wire Wire Line
+	3350 2400 3350 2550
+Wire Wire Line
+	4600 2200 3100 2200
+Wire Wire Line
+	3100 2050 3100 2350
+Connection ~ 3100 2200
+Text Notes 14600 10950 2    60   ~ 12
+NIGUN - 1500-3000MHz RF downconverter for SDR
+Text Notes 13550 11050 2    60   ~ 12
+02/10/2016
 $EndSCHEMATC
