File: Schematics/_saved_Nigun.sch (KiCad schematic (older format))
At the start: 146 parts, among them J1 USB-MICRO-B, J2 RF_INPUT, J3 RF_OUTPUT, P1 CONN_02X04, P2 CONN_SWD, SW1 SW_PUSH_SMALL_H, T1 TC1-1-43A+, T2 TC4-1W+, U1 STF202, U2 SKY13351, U3 MIC5504-3.3YM5-TR, U4 AP7365-WG-7, U5 LP0805A0881AS, U6 ADRF6612, U7 FOX924B-16.000, U8 SKY13373, U9 ATSAMD21E

Commit message: Finished schematics
Parts:
- C1, C10, C11, C12, C13, C14, C15, C16, C17, C18, C19, C2, C20, C21, C22, C23, C24, C25, C26, C27, C28, C29, C3, C30, C31, C32, C33, C34, C35, C36, C37, C38, C39, C4, C40, C41, C42, C43, C44, C45, C46, C47, C48, C49, C5, C50, C51, C52, C53, C54, C55, C56, C57, C58, C59, C6, C60, C61, C62, C63, C64, C65, C66, C67, C68, C69, C7, C70, C71, C72, C73, C74, C75, C76, C77, C78, C79, C8, C80, C81, C82, C83, C84, C85, C86, C87, C88, C89, C9: footprint Capacitors_SMD:C_0805_HandSoldering -> Capacitors_SMD:C_0402
- D1: symbol D_Schottky_Small -> D_Schottky_Small-RESCUE-Nigun
- J2, J3: footprint gsg-modules:SMA-EDGE -> adafruit:SMA_EDGELAUNCH
- R1, R10, R11, R12, R13, R14, R15, R16, R17, R18, R19, R2, R20, R21, R22, R23, R24, R25, R26, R27, R28, R29, R3, R30, R31, R32, R4, R5, R6, R7, R8, R9: footprint Resistors_SMD:R_0805_HandSoldering -> Resistors_SMD:R_0402
- U3: footprint TO_SOT_Packages_SMD:SOT-223 -> TO_SOT_Packages_SMD:SOT-23-5
