File: Schematics/Nigun.sch (KiCad schematic (older format))
At the start: 41 parts, among them J1 RF_INPUT, U1 ADRF6612, U2 SKY13373

Commit message: Schematics
Parts:
- added C? (x10): 100pF, symbol C
- added C? (x18): 10uF, symbol C
- added C? (x8): 10pF, symbol C
- added C? (x8): 0.1uF, symbol C
- added C? (x3): 150pF, symbol C
- added C?: 1000pF, symbol C
- added L? (x2): 330nH, symbol L_Small
- added R?: 50, symbol R
- added R?: 2k, symbol R
- added T?: TC1-1-43A+, symbol TC1-1-43A+
- added T?: TC4-1W+, symbol TC4-1W+
- U1: footprint (none) -> ADRF6612_LFCSP48:LFCSP48
Connections:
- net labels added: 6612IN_RFIN, 6612OUT_MUXOUT, VCC
- wire segments 66 -> 148
Other:
- note added: "02/10/2016"
- note added: "GIT"
- note added: "NIGUN - 1500-3000MHz RF downconverter for SDR"
- moved on the sheet: C1, C2, C3, C4, C5, C?, J1, J?, R?, T?, U1, U2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

Commit message: Schematics update
Parts:
- added C44, C46, C53: 1000pF, symbol C
- added C?: 10uF, symbol C
- added C?: 100pF, symbol C
- added C? (x2): 1uF, symbol C
- added D?: D_Schottky_Small, symbol D_Schottky_Small
- added J?: USB-MICRO-B, symbol USB-MICRO-B
- added R10, R11, R9: 50, symbol R
- added U?: MIC5504-3.3YM5-TR, SOT-223, symbol MIC5504-3.3YM5-TR
- added U?: AP7365-WG-7, symbol AP7365-WG-7
- added U?: SAMD20E17A-A, TQFP32, symbol SAMD20E17A-A
- added U?: ECS-TXO-5032-200-TR, symbol ECS-TXO-5032-200-TR
- gave numbers to parts that had none: 87
Connections:
- net labels added: +5V, ADRF_CSNOT, ADRF_REFIN, ADRF_SCLK, ADRF_SDIO, OUTSW_V1, OUTSW_V2, OUTSW_VDD, SWIN_VCTL1, SWIN_VCTL2, VCC_3.3V, VCC_3.7V
- net labels removed: 6612IN_RFIN, RF_IN_SW_VCTL1, RF_IN_SW_VCTL2, VCC
- wire segments 148 -> 181
- no-connect marks 0 -> 4
Other:
- moved on the sheet: C1, C10, C11, C12, C13, C14, C15, C16, C17, C18, C19, C2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

Commit message: Almost finished schematics, based on ATSAMD20E MCU
Parts:
- removed U?: ECS-TXO-5032-200-TR, symbol ECS-TXO-5032-200-TR
- added C80, C82, C86: 1uF, symbol C
- added C85, C88: 10uF, symbol C
- added C87, C89: 100nF, symbol C
- added D2, D3, D4: blue_led, symbol Led_Small
- added D5: green_led, symbol Led_Small
- added L3: 10uH, symbol L_Small
- added P1: CONN_02X04, symbol CONN_02X04
- added P2: CONN_02X03, symbol CONN_02X03
- added R12: 3.92K, symbol R
- added R13: 2K, symbol R
- added R14: 10k, symbol R
- added R15, R16: 68, symbol R
- added R17: 10K, symbol R
- added R18: 330, symbol R
- added R19, R20, R21: 1k, symbol R
- added SW1: SW_PUSH_SMALL_H, symbol SW_PUSH_SMALL_H
- added U7: FOX924B-16.000, symbol FOX924B-16.000
- U8: renamed from U?; footprint TQFP32 -> samd20e17a:QFN50P500X500X100-33N
- gave numbers to parts that had none: 8
Connections:
- net labels added: RESET, USB_DM, USB_DP, V_EXT
- net labels removed: OUTSW_VDD
- wire segments 181 -> 341
- no-connect marks 4 -> 8
Other:
- note added: "CLK"
- note added: "Debug pads"
- note added: "MCU"
- note added: "MCU \nProgramming \nport"
- note added: "MISO"
- note added: "MOSI"
- note added: "Power supply and USB connection"
- note added: "Signal Input"
- moved on the sheet: C41, C42, C79, C81, J3, T2, U2, U5, U6

Commit message: Finished schematics
Parts:
- removed C11, C21, C22: 100pF, symbol C
- removed C85, C88: 10uF, symbol C
- removed C86: 1uF, symbol C
- removed C87, C89: 100nF, symbol C
- removed J2: SMA, SMA, symbol SMA
- removed P2: CONN_02X03, symbol CONN_02X03
- removed R14: 10k, symbol R
- removed R15, R16: 68, symbol R
- removed R17: 10K, symbol R
- removed T1: TC1-1-43A+, symbol TC1-1-43A+
- removed U8: SAMD20E17A-A, samd20e17a:QFN50P500X500X100-33N, symbol SAMD20E17A-A
- added C32, C33: 1000pF, Capacitors_SMD:C_0805_HandSoldering, symbol C
- added C71, C88: 10uF, Capacitors_SMD:C_0805_HandSoldering, symbol C_Small
- added C78, C87, C89: 100nF, Capacitors_SMD:C_0805_HandSoldering, symbol C_Small
- added C86: 1uF, Capacitors_SMD:C_0805_HandSoldering, symbol C_Small
- added P2: CONN_SWD, gsg-modules:HEADER-2x5, symbol CONN_SWD
- added R10, R11: 50, Resistors_SMD:R_0805_HandSoldering, symbol R
- added R17, R20, R21, R22, R23, R24, R25, R26, R27, R28, R29: 0, Resistors_SMD:R_0805_HandSoldering, symbol R_Small
- added R18: 10k, Resistors_SMD:R_0805_HandSoldering, symbol R_Small
- added R31: 10k, Resistors_SMD:R_0805_HandSoldering, symbol R
- added U1: STF202, hack-footprints:TSOP-6, symbol STF202
- added U9: ATSAMD21E, QFN32:QFN32, symbol ATSAMD21E
- C1, L1, L2, L3: footprint (none) -> Capacitors_SMD:C_0805_HandSoldering
- C10: renamed from C79; footprint (none) -> Capacitors_SMD:C_0805_HandSoldering
- C11: renamed from C13; footprint (none) -> Capacitors_SMD:C_0805_HandSoldering
- C12: renamed from C14; footprint (none) -> Capacitors_SMD:C_0805_HandSoldering
- C13: renamed from C15; footprint (none) -> Capacitors_SMD:C_0805_HandSoldering
- C14: renamed from C80; footprint (none) -> Capacitors_SMD:C_0805_HandSoldering
- C15: renamed from C16; footprint (none) -> Capacitors_SMD:C_0805_HandSoldering
- C16: renamed from C17; footprint (none) -> Capacitors_SMD:C_0805_HandSoldering
- C17: renamed from C18; footprint (none) -> Capacitors_SMD:C_0805_HandSoldering
- C18: renamed from C19; footprint (none) -> Capacitors_SMD:C_0805_HandSoldering
- C19: renamed from C20; footprint (none) -> Capacitors_SMD:C_0805_HandSoldering
- C2: renamed from C6; footprint (none) -> Capacitors_SMD:C_0805_HandSoldering
- C20: renamed from C81; footprint (none) -> Capacitors_SMD:C_0805_HandSoldering
- C21: renamed from C23; footprint (none) -> Capacitors_SMD:C_0805_HandSoldering
- C22: renamed from C24; footprint (none) -> Capacitors_SMD:C_0805_HandSoldering
- C23: renamed from C25; footprint (none) -> Capacitors_SMD:C_0805_HandSoldering
- C24: renamed from C26; footprint (none) -> Capacitors_SMD:C_0805_HandSoldering
- C25: renamed from C27; footprint (none) -> Capacitors_SMD:C_0805_HandSoldering
- C26: renamed from C82; footprint (none) -> Capacitors_SMD:C_0805_HandSoldering
- C27: renamed from C28; footprint (none) -> Capacitors_SMD:C_0805_HandSoldering
- C28: renamed from C29; footprint (none) -> Capacitors_SMD:C_0805_HandSoldering
- C29: renamed from C30; footprint (none) -> Capacitors_SMD:C_0805_HandSoldering
- C3: renamed from C7; footprint (none) -> Capacitors_SMD:C_0805_HandSoldering
- C30: renamed from C31; footprint (none) -> Capacitors_SMD:C_0805_HandSoldering
- C31: renamed from C32; footprint (none) -> Capacitors_SMD:C_0805_HandSoldering
- C34: renamed from C33; footprint (none) -> Capacitors_SMD:C_0805_HandSoldering
- C35: renamed from C34; footprint (none) -> Capacitors_SMD:C_0805_HandSoldering
- C36: renamed from C35; footprint (none) -> Capacitors_SMD:C_0805_HandSoldering
- C37: renamed from C36; footprint (none) -> Capacitors_SMD:C_0805_HandSoldering
- C38: renamed from C37; footprint (none) -> Capacitors_SMD:C_0805_HandSoldering
- C39: renamed from C38; footprint (none) -> Capacitors_SMD:C_0805_HandSoldering
- C4: renamed from C8; footprint (none) -> Capacitors_SMD:C_0805_HandSoldering
- C40: renamed from C39; footprint (none) -> Capacitors_SMD:C_0805_HandSoldering
- C41: renamed from C40; footprint (none) -> Capacitors_SMD:C_0805_HandSoldering
- C42: renamed from C83; footprint (none) -> Capacitors_SMD:C_0805_HandSoldering
- C43: renamed from C41; footprint (none) -> Capacitors_SMD:C_0805_HandSoldering
- C44: renamed from C42; footprint (none) -> Capacitors_SMD:C_0805_HandSoldering
- C45: renamed from C84; footprint (none) -> Capacitors_SMD:C_0805_HandSoldering
- C46: renamed from C43; footprint (none) -> Capacitors_SMD:C_0805_HandSoldering
- C47: renamed from C44; footprint (none) -> Capacitors_SMD:C_0805_HandSoldering
- C48: renamed from C45; footprint (none) -> Capacitors_SMD:C_0805_HandSoldering
- C49: renamed from C46; footprint (none) -> Capacitors_SMD:C_0805_HandSoldering
- C5: renamed from C9; footprint (none) -> Capacitors_SMD:C_0805_HandSoldering
- C50: renamed from C47; footprint (none) -> Capacitors_SMD:C_0805_HandSoldering
- C51: renamed from C48; footprint (none) -> Capacitors_SMD:C_0805_HandSoldering
- C52: renamed from C49; footprint (none) -> Capacitors_SMD:C_0805_HandSoldering
- C53: renamed from C50; footprint (none) -> Capacitors_SMD:C_0805_HandSoldering
- C54: renamed from C51; footprint (none) -> Capacitors_SMD:C_0805_HandSoldering
- C55: renamed from C52; footprint (none) -> Capacitors_SMD:C_0805_HandSoldering
- C56: renamed from C53; footprint (none) -> Capacitors_SMD:C_0805_HandSoldering
- C57: renamed from C54; footprint (none) -> Capacitors_SMD:C_0805_HandSoldering
- C58: renamed from C55; footprint (none) -> Capacitors_SMD:C_0805_HandSoldering
- C59: renamed from C4; footprint (none) -> Capacitors_SMD:C_0805_HandSoldering
- C6: renamed from C10; footprint (none) -> Capacitors_SMD:C_0805_HandSoldering
- C60: renamed from C5; footprint (none) -> Capacitors_SMD:C_0805_HandSoldering
- C61: renamed from C56; footprint (none) -> Capacitors_SMD:C_0805_HandSoldering
- C62: renamed from C57; footprint (none) -> Capacitors_SMD:C_0805_HandSoldering
- C63: renamed from C58; footprint (none) -> Capacitors_SMD:C_0805_HandSoldering
- C64: renamed from C59; footprint (none) -> Capacitors_SMD:C_0805_HandSoldering
- C65: renamed from C60; footprint (none) -> Capacitors_SMD:C_0805_HandSoldering
- C66: renamed from C61; footprint (none) -> Capacitors_SMD:C_0805_HandSoldering
- C67: renamed from C62; footprint (none) -> Capacitors_SMD:C_0805_HandSoldering
- C68: renamed from C63; footprint (none) -> Capacitors_SMD:C_0805_HandSoldering
- C69: renamed from C64; footprint (none) -> Capacitors_SMD:C_0805_HandSoldering
- C7: renamed from C3; footprint (none) -> Capacitors_SMD:C_0805_HandSoldering
- C70: renamed from C65; footprint (none) -> Capacitors_SMD:C_0805_HandSoldering
- C72: renamed from C66; footprint (none) -> Capacitors_SMD:C_0805_HandSoldering
- C73: renamed from C67; footprint (none) -> Capacitors_SMD:C_0805_HandSoldering
- C74: renamed from C68; footprint (none) -> Capacitors_SMD:C_0805_HandSoldering
- C75: renamed from C69; footprint (none) -> Capacitors_SMD:C_0805_HandSoldering
- C76: renamed from C70; footprint (none) -> Capacitors_SMD:C_0805_HandSoldering
- C77: renamed from C71; footprint (none) -> Capacitors_SMD:C_0805_HandSoldering
- C79: renamed from C72; footprint (none) -> Capacitors_SMD:C_0805_HandSoldering
- C8: renamed from C2; footprint (none) -> Capacitors_SMD:C_0805_HandSoldering
- C80: renamed from C73; footprint (none) -> Capacitors_SMD:C_0805_HandSoldering
- C81: renamed from C74; footprint (none) -> Capacitors_SMD:C_0805_HandSoldering
- C82: renamed from C75; footprint (none) -> Capacitors_SMD:C_0805_HandSoldering
- C83: renamed from C76; footprint (none) -> Capacitors_SMD:C_0805_HandSoldering
- C84: renamed from C77; footprint (none) -> Capacitors_SMD:C_0805_HandSoldering
- C85: renamed from C78; footprint (none) -> Capacitors_SMD:C_0805_HandSoldering
- C9: renamed from C12; footprint (none) -> Capacitors_SMD:C_0805_HandSoldering
- D1: footprint (none) -> Footprints:DO-214AA-SMB
- D2: value blue_led -> Red; footprint (none) -> Footprints:LED_kingsbright
- D3: renamed from D5; value green_led -> Green; footprint (none) -> Footprints:LED_kingsbright
- D4: renamed from D3; value blue_led -> Blue; footprint (none) -> Footprints:LED_kingsbright
- D5: renamed from D4; value blue_led -> Red; footprint (none) -> Footprints:LED_kingsbright
- J1: renamed from J4; footprint (none) -> gsg-modules:USB-MICROB-FCI-10103592-EXT
- J2: renamed from J1; footprint SMA -> adafruit:SMA_EDGELAUNCH
- J3: value SMA -> RF_OUTPUT; footprint SMA -> adafruit:SMA_EDGELAUNCH
- P1: footprint (none) -> gsg-modules:HEADER-2x4
- R1, R2, R3, R4, R5: footprint (none) -> Resistors_SMD:R_0805_HandSoldering
- R12: renamed from R7; footprint (none) -> Resistors_SMD:R_0805_HandSoldering
- R13: renamed from R9; footprint (none) -> Resistors_SMD:R_0805_HandSoldering
- R14: renamed from R10; footprint (none) -> Resistors_SMD:R_0805_HandSoldering
- R15: renamed from R11; footprint (none) -> Resistors_SMD:R_0805_HandSoldering
- R16: renamed from R21; value 1k -> 330; footprint (none) -> Resistors_SMD:R_0805_HandSoldering
- R19: renamed from R8; value 2k -> 330; footprint (none) -> Resistors_SMD:R_0805_HandSoldering
- R30: renamed from R20; value 1k -> 330; footprint (none) -> Resistors_SMD:R_0805_HandSoldering
- R32: renamed from R18; footprint (none) -> Resistors_SMD:R_0805_HandSoldering
- R6: renamed from R19; value 1k -> 330; footprint (none) -> Resistors_SMD:R_0805_HandSoldering
- R7: renamed from R12; footprint (none) -> Resistors_SMD:R_0805_HandSoldering
- R8: renamed from R13; footprint (none) -> Resistors_SMD:R_0805_HandSoldering
- R9: renamed from R6; footprint (none) -> Resistors_SMD:R_0805_HandSoldering
- SW1: footprint (none) -> Footprints:Tactile_SW
- T1: renamed from T2; footprint (none) -> Footprints:AT224-1A
- T2: renamed from T3; footprint (none) -> Footprints:AT224-1A
- U2: renamed from U3; footprint (none) -> gsg-modules:SKY13351-378LF
- U3: renamed from U5; footprint SOT-223 -> TO_SOT_Packages_SMD:SOT-23-5
- U4: renamed from U6; footprint (none) -> gsg-modules:SOT25
- U5: renamed from U4; value LP0805A1119AS -> LP0805A0881AS; footprint (none) -> Footprints:CP_0805
- U7: footprint (none) -> Footprints:FOX924
- U8: renamed from U2; footprint (none) -> Housings_DFN_QFN:QFN-12-1EP_3x3mm_Pitch0.5mm
- renumbered U1 to U6
Connections:
- net labels added: !RESET, ADRF_MUXOUT, ADRF_VTUNE, IN_SW_VCTL1, IN_SW_VCTL2, MCU_VDDIN, OUT_SW_V1, OUT_SW_V2, SWDCLK, SWDIO, TCXO_OUT, USB_D+, USB_D-
- net labels removed: +5V, 6612OUT_MUXOUT, CPOUT, OUTSW_V1, OUTSW_V2, RESET, SWIN_VCTL1, SWIN_VCTL2, USB_DM, USB_DP, VTUNE
- wire segments 341 -> 217
- no-connect marks 8 -> 4
Other:
- note added: "DEBUG PINS"
- note added: "NIGUN (MELODY)"
- note added: "NIGUN (MELODY)\n1500-3000MHz RF Down-converter"
- note added: "SWD DEBUG CONNECTOR"
- note added: "TCXO"
- note removed: "CLK"
- note removed: "Debug pads"
- note removed: "MCU \nProgramming \nport"
- note removed: "NIGUN - 1500-3000MHz RF downconverter for SDR"
- moved on the sheet: C10, C14, C20, C26, D2, D3, D4, D5, L3, P1, R16, R19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

Commit message: replaced 45deg bent RF traces with curvy traces
Parts:
- C1, C10, C11, C12, C13, C14, C15, C16, C17, C18, C19, C2, C20, C21, C22, C23, C24, C25, C26, C27, C28, C29, C3, C30, C31, C32, C33, C34, C35, C36, C37, C38, C39, C4, C40, C41, C42, C43, C44, C45, C46, C47, C48, C49, C5, C50, C51, C52, C53, C54, C55, C56, C57, C58, C59, C6, C60, C61, C62, C63, C64, C65, C66, C67, C68, C69, C7, C70, C71, C72, C73, C74, C75, C76, C77, C78, C79, C8, C80, C81, C82, C83, C84, C85, C86, C87, C88, C89, C9: footprint Capacitors_SMD:C_0805_HandSoldering -> Capacitors_SMD:C_0402
- D1: symbol D_Schottky_Small -> D_Schottky_Small-RESCUE-Nigun
- R1, R10, R11, R12, R13, R14, R15, R16, R17, R18, R19, R2, R20, R21, R22, R23, R24, R25, R26, R27, R28, R29, R3, R30, R31, R32, R4, R5, R6, R7, R8, R9: footprint Resistors_SMD:R_0805_HandSoldering -> Resistors_SMD:R_0402

Commit message: PCB design update - finished RF traces and 2 sides of 6612
Parts:
- added C47, C52: 150pF, Capacitors_SMD:C_0402, symbol C
- D2, D3, D4, D5: symbol Led_Small -> Led_Small-RESCUE-Nigun
- L1, L2: footprint Capacitors_SMD:C_0805_HandSoldering -> Capacitors_SMD:C_0402
- renumbered C47 to C48, C48 to C49, C49 to C50, C50 to C51, C51 to C53, C52 to C54, C53 to C55, C54 to C56, C55 to C57, C56 to C58, C57 to C59, C58 to C60, C59 to C61, C60 to C62, C61 to C63, C62 to C64, C63 to C65, C64 to C66, C65 to C67, C66 to C68, C67 to C69, C68 to C70, C69 to C71, C70 to C72, C71 to C73, C72 to C74, C73 to C75, C74 to C76, C75 to C77, C76 to C78, C77 to C79, C78 to C80, C79 to C81, C80 to C82, C81 to C83, C82 to C84, C83 to C85, C84 to C86, C85 to C87, C86 to C88, C87 to C89, C88 to C90, C89 to C91
Connections:
- net Earth: now also T1.4, C47.2, C52.1; no longer T1.6
- net VCC_3.7V: now also C47.1, C52.2
- net LOOUT+: now reaches C43.1, U6.13 (LOOUT+)
- net LOOUT-: now reaches C44.1, U6.14 (LOOUT-)
- net IFOUT2+: now reaches C48.1, U6.22 (IFOUT2+)
- net IFOUT2-: now reaches C50.1, U6.23 (IFOUT2-)
- net IFOUT1-: now reaches L2.2, U6.38 (IFOUT-)
- net IFOUT1-: now also C54.2; no longer C53.2
- net IFOUT1+: now reaches L1.2, U6.39 (IFOUT+)
- net IFOUT1+: now also C53.2; no longer C54.2
- net EXTVCOIN+: now reaches C32.1, U6.4 (EXTVCOIN+)
- net EXTVCOIN-: now reaches C33.1, U6.5 (EXTVCOIN-)
- net at U8.1 (J1): now also T1.6; no longer T2.6
- net at U8.3 (J3): now also T2.6; no longer T1.4
- net TC1IN+: now reaches C43.2, T1.1
- net TC1IN-: now reaches C44.2, T1.3
- net TC4IN+: now reaches C53.1, T2.1
- net TC4IN-: now reaches C54.1, T2.3

Commit message: Changed ESD protection IC for USB bus
Parts:
- removed U1: STF202, hack-footprints:TSOP-6, symbol STF202
- added D6: PRTR5V0U2X, SOT143B, symbol PRTR5V0U2X
Connections:
- net Earth: now also D6.1 (P$1)
- net USB_D+: now also J1.3 (D+), D6.3 (P$3)
- net USB_D-: now also J1.2 (D-), D6.2 (P$2)
- net at J1.1 (VBUS), R1.1: now also D6.4 (P$4)
Changed lines of the file:
@@
 F 0 "J1" H 900 1250 60  0000 C CNN
 F 1 "USB-MICRO-B" H 900 600 60  0000 C CNN
-F 2 "gsg-modules:USB-MICROB-FCI-10103592-EXT" H 900 950 60  0000 C CNN
+F 2 "gsg-modules:USB-MICROB-FCI-10103592-EXT" H 850 500 60  0001 C CNN
 F 3 "" H 900 950 60  0000 C CNN
 	1    900  950
@@
 	1    0    0    -1
 $EndComp
-Text GLabel 2150 2350 2    39   BiDi ~ 0
+Text GLabel 1950 1850 2    39   BiDi ~ 0
 USB_D+
-Text GLabel 2150 2450 2    39   BiDi ~ 0
+Text GLabel 1950 1950 2    39   BiDi ~ 0
 USB_D-
 $Comp
@@
 	0    -1   -1   0
 $EndComp
-$Comp
-L STF202 U1
-U 1 1 586C0C97
-P 1750 2100
-F 0 "U1" H 1500 2150 40  0000 C CNB
-F 1 "STF202" H 1750 2150 40  0000 C CNB
-F 2 "hack-footprints:TSOP-6" H 1400 2050 60  0000 C CNN
-F 3 "" H 1500 2150 60  0000 C CNN
-F 4 "STF202-22T1G" H 1750 2200 60  0000 C CNN "manf#"
-	1    1750 2100
-	1    0    0    -1
-$EndComp
 Connection ~ 12650 5800
 Wire Wire Line
@@
 	14550 5500 14550 4650
 Wire Wire Line
-	1150 1150 1950 1150
-Wire Wire Line
 	5600 2650 5600 3500
 Wire Wire Line
@@
 Connection ~ 5600 2650
 Wire Wire Line
-	1150 1050 1300 1050
-Wire Wire Line
-	1300 1050 1300 2350
-Wire Wire Line
-	1300 2350 1350 2350
-Wire Wire Line
-	1350 1150 1350 2250
-Connection ~ 1350 1150
-Wire Wire Line
-	1150 950  1250 950
-Wire Wire Line
-	1250 950  1250 2450
-Wire Wire Line
-	1250 2450 1350 2450
+	1150 1050 1600 1050
+Wire Wire Line
+	1150 950  1800 950
 $Comp
 L Earth #PWR065
 U 1 1 586C4520
-P 2150 2250
-F 0 "#PWR065" H 2150 2000 50  0001 C CNN
-F 1 "Earth" H 2150 2100 50  0001 C CNN
-F 2 "" H 2150 2250 50  0000 C CNN
-F 3 "" H 2150 2250 50  0000 C CNN
-	1    2150 2250
-	0    -1   -1   0
+P 1300 2650
+F 0 "#PWR065" H 1300 2400 50  0001 C CNN
+F 1 "Earth" H 1300 2500 50  0001 C CNN
+F 2 "" H 1300 2650 50  0000 C CNN
+F 3 "" H 1300 2650 50  0000 C CNN
+	1    1300 2650
+	1    0    0    -1
 $EndComp
 $Comp
@@
 Wire Wire Line
 	8600 9100 7400 9100
+Text Label 1250 950  0    60   ~ 0
+D+
+Text Label 1300 1050 0    60   ~ 0
+D-
+$Comp
+L PRTR5V0U2X D6
+U 1 1 589FED3C
+P 1500 2350
+F 0 "D6" H 1400 2054 50  0000 L CNN
+F 1 "PRTR5V0U2X" H 1400 1944 50  0000 L CNN
+F 2 "SOT143B" H 1500 2350 50  0001 L CNN
+F 3 "NXP Semiconductors" H 1200 2800 50  0001 L CNN
+F 4 "SOT-143 NXP Semiconductors" H 1000 2900 50  0001 L CNN "Package"
+F 5 "0.38 USD" H 1500 2350 50  0001 L CNN "Price"
+F 6 "PRTR5V0U2X" H 1500 2350 50  0001 L CNN "MP"
+F 7 "Good" H 1500 2350 50  0001 L CNN "Availability"
+F 8 "DIODE, TVS, DUAL, SOT-143B; Diode Type: TVS, Bidirectional; Voltage, Stand-off: 5.5V; Voltage, Vbr: 9V; Termination T..." H -450 1800 50  0001 L CNN "Description"
+	1    1500 2350
+	1    0    0    -1
+$EndComp
+Wire Wire Line
+	1300 2050 1300 1150
+Wire Wire Line
+	1150 1150 1950 1150
+Connection ~ 1300 1150
+Wire Wire Line
+	1600 1050 1600 2050
+Wire Wire Line
+	1800 950  1800 2050
+Wire Wire Line
+	1950 1850 1800 1850
+Connection ~ 1800 1850
+Wire Wire Line
+	1950 1950 1600 1950
+Connection ~ 1600 1950
 $EndSCHEMATC

Commit message: Place and route updates
Parts:
- removed C2, C21: 10uF, Capacitors_SMD:C_0402, symbol C
- D6: footprint SOT143B -> Footprints:SOT143B
- J1: footprint gsg-modules:USB-MICROB-FCI-10103592-EXT -> Footprints:FRAMATOME_10118194-0001LF
Changed lines of the file:
@@
 GIT
-$Comp
-L C C21
-U 1 1 583E122C
-P 4200 6300
-F 0 "C21" H 4225 6400 50  0000 L CNN
-F 1 "10uF" H 4225 6200 50  0000 L CNN
-F 2 "Capacitors_SMD:C_0402" H 4238 6150 50  0001 C CNN
-F 3 "" H 4200 6300 50  0000 C CNN
-	1    4200 6300
-	1    0    0    -1
-$EndComp
 $Comp
 L C C27
@@
 F 3 "" H 5050 7450 50  0000 C CNN
 	1    5050 7450
-	1    0    0    -1
-$EndComp
-$Comp
-L C C2
-U 1 1 583F48BA
-P 2150 4300
-F 0 "C2" H 2175 4400 50  0000 L CNN
-F 1 "10uF" H 2175 4200 50  0000 L CNN
-F 2 "Capacitors_SMD:C_0402" H 2188 4150 50  0001 C CNN
-F 3 "" H 2150 4300 50  0000 C CNN
-	1    2150 4300
 	1    0    0    -1
 $EndComp
@@
 F 0 "J1" H 900 1250 60  0000 C CNN
 F 1 "USB-MICRO-B" H 900 600 60  0000 C CNN
-F 2 "gsg-modules:USB-MICROB-FCI-10103592-EXT" H 850 500 60  0001 C CNN
+F 2 "Footprints:FRAMATOME_10118194-0001LF" H 850 500 60  0001 C CNN
 F 3 "" H 900 950 60  0000 C CNN
 	1    900  950
@@
 Connection ~ 4850 3500
 Connection ~ 5600 2650
-Wire Wire Line
-	1150 1050 1600 1050
-Wire Wire Line
-	1150 950  1800 950
 $Comp
 L Earth #PWR065
@@
 F 0 "D6" H 1400 2054 50  0000 L CNN
 F 1 "PRTR5V0U2X" H 1400 1944 50  0000 L CNN
-F 2 "SOT143B" H 1500 2350 50  0001 L CNN
+F 2 "Footprints:SOT143B" H 1500 2350 50  0001 L CNN
 F 3 "NXP Semiconductors" H 1200 2800 50  0001 L CNN
 F 4 "SOT-143 NXP Semiconductors" H 1000 2900 50  0001 L CNN "Package"
@@
 $EndComp
 Wire Wire Line
-	1300 2050 1300 1150
-Wire Wire Line
 	1150 1150 1950 1150
 Connection ~ 1300 1150
 Wire Wire Line
+	1800 950  1800 2050
+Wire Wire Line
+	1150 950  1800 950
+Wire Wire Line
+	1150 1050 1600 1050
+Wire Wire Line
 	1600 1050 1600 2050
 Wire Wire Line
-	1800 950  1800 2050
+	1950 1950 1600 1950
+Connection ~ 1600 1950
 Wire Wire Line
 	1950 1850 1800 1850
 Connection ~ 1800 1850
 Wire Wire Line
-	1950 1950 1600 1950
-Connection ~ 1600 1950
+	1300 2050 1300 1150
 $EndSCHEMATC
