File: Schematics/_autosave-Nigun.kicad_pcb (KiCad board)
At the start: 4 copper layers, 53.9 x 50.8 mm, 146 parts, among them J1 USB-MICRO-B, J2 RF_INPUT, J3 RF_OUTPUT, P1 CONN_02X04, P2 CONN_SWD, SW1 SW_PUSH_SMALL_H, T1 TC1-1-43A+, T2 TC4-1W+, U2 SKY13351, U3 MIC5504-3.3YM5-TR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

Commit message: Finished front layer
Routing:
- net Net-(C56-Pad2): track 2.97 -> 4.20 mm
Changed lines of the file:
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@@
     (thickness 1.6)
     (drawings 9)
-    (tracks 1346)
+    (tracks 1347)
     (zones 0)
     (modules 146)
@@
   (page A4)
   (layers
-    (0 Front signal)
-    (1 VCC power)
+    (0 Front signal hide)
+    (1 VCC power hide)
     (2 GND power)
-    (31 Back signal)
-    (33 F.Adhes user)
-    (35 F.Paste user)
+    (31 Back signal hide)
+    (33 F.Adhes user hide)
+    (35 F.Paste user hide)
     (37 F.SilkS user hide)
     (39 F.Mask user hide)
@@
     (43 Eco2.User user)
     (44 Edge.Cuts user)
-    (45 Margin user)
-    (47 F.CrtYd user)
+    (45 Margin user hide)
+    (47 F.CrtYd user hide)
     (49 F.Fab user hide)
   )
@@
   (gr_line (start 169.3545 43.688) (end 169.3545 91.44) (angle 90) (layer Edge.Cuts) (width 0.2))
   (gr_line (start 116.84 42.291) (end 167.64 42.291) (angle 90) (layer Edge.Cuts) (width 0.2))
-  (segment (start 135.717736 54.074291) (end 135.72172 54.070307) (width 0.3302) (layer Back) (net 0))
   (segment (start 127.35306 54.4322) (end 126.7968 54.4449) (width 0.1524) (layer Front) (net 1))
   (segment (start 125.6792 54.4322) (end 126.7968 54.4449) (width 0.4318) (layer Front) (net 1))
@@
   (segment (start 155.94466 44.44238) (end 155.922034 44.465006) (width 0.4318) (layer Front) (net 24))
   (segment (start 156.188734 46.195933) (end 156.18968 46.19688) (width 0.4318) (layer Front) (net 24))
+  (segment (start 134.8144 55.6514) (end 134.8144 54.441) (width 0.3302) (layer Front) (net 25))
+  (segment (start 134.8144 54.441) (end 134.8056 54.4322) (width 0.3302) (layer Front) (net 25))
   (segment (start 137.7882 55.6792) (end 134.8144 55.6514) (width 0.3302) (layer Front) (net 25))
   (segment (start 138.2882 55.7042) (end 138.277176 55.015976) (width 0.3302) (layer Front) (net 26))
